File: main_board/power.kicad_sch (KiCad schematic)
At the start: 44 parts, among them J10 Conn_01x02, J11 B2B-XH-A(LF)(SN), J12 B2B-XH-A(LF)(SN), J13 B2B-XH-A(LF)(SN), J16 B4B-ZR(LF)(SN), J9 MJ-179PH, Q5 DMT6008LFG, Q6 DMT6008LFG, Q7 DTC114E, Q8 DTC114E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

Commit message: アートワークひととおり完成
Parts:
- removed J13: B2B-XH-A(LF)(SN), Connector_PinHeader_2.54mm:PinHeader_1x02_P2.54mm_Vertical, symbol Connector_Generic:Conn_01x02
- J10, J11, J12: footprint Connector_PinHeader_2.54mm:PinHeader_1x02_P2.54mm_Vertical -> Connector_JST:JST_XH_B2B-XH-AM_1x02_P2.50mm_Vertical
