File: main_board/main_board.kicad_sch (KiCad schematic)
At the start: 75 parts, among them J1 Conn_01x02, J2 Conn_01x02, J3 2.54mm PinHeader, J4 EncSide, J5 B6B-ZR, J6 2.54mm PinHeader, J7 EncSide, J8 B6B-ZR, Q1 IRLML6344, Q2 IRLML6344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

Commit message: アートワークひととおり完成
Parts:
- added C18, C19: CC0603KRX7R9BB104, Capacitor_SMD:C_0603_1608Metric, symbol Device:C_Small
Connections:
- net +3V3: now also C18.1, C19.1
- net GND: now also C18.2, C19.2

Commit message: 12/18 基板発注
Parts:
- removed C15, C16: CC0603KRX7R9BB104, Capacitor_SMD:C_0603_1608Metric, symbol Device:C_Small
- removed H10, H5, H6, H7, H8, H9: M2 mounting hole, MountingHole:MountingHole_2.2mm_M2, symbol Mechanical:MountingHole
- removed J4, J7: EncSide, Library:EncoderPad, symbol Connector:Conn_01x06_Male
- removed U10, U9: AS5047D, Package_SO:TSSOP-14_4.4x5mm_P0.65mm, symbol Sensor_Magnetic:AS5047D
- C18, C19: value CC0603KRX7R9BB104 -> CL10A105KB8NNNC
Connections:
- net GND: now also U2.11 (PGND), U5.11 (PGND), U6.40 (GND), U6.41 (GND)
- no-connect marks 31 -> 17
Other:
- moved on the sheet: J5, J8
