File: sub_boards/sub_boards/sub_boards.kicad_sch (KiCad schematic)
At the start: 16 parts, among them J1 Raspberry_Pi_5, J3 2.54mm PinHeader, J4 2.54mm PinHeader, Q1 ST-1KL3A, Q2 ST-1KL3A, Q3 ST-1KL3A, Q4 ST-1KL3A, SW1 TVBP06-B043CB-B, SW2 TVBP06-B043CB-B, SW3 TVBP06-B043CB-B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

Commit message: サブ基板アートワーク完了
Signed-off-by: Kazuki Iida <elkel53930@gmail.com>
Parts:
- added H1, H2: MountingHole, Library:M2.6 Mounting Hole, symbol Mechanical:MountingHole
Connections:
- net BTN_DOWN: now also J1.7 (GPCLK0/GPIO04), SW1.1; no longer J1.35 (GPIO19/SPI1_MISO/PCM_FS), SW2.1
- net BTN_LEFT: now also J1.3 (SDA_I2C1/GPIO02), SW4.1; no longer J1.38 (GPIO20/SPI1_MOSI/PCM_DIN/PWM1), SW3.1
- net BTN_RIGHT: now also J1.5 (SCL_I2C1/GPIO03), SW3.1; no longer J1.36 (GPIO16/SPI1_~{CE2}), SW4.1
- net BTN_UP: now also J1.11 (GPIO17/SPI1_~{CE1}), SW2.1; no longer J1.37 (GPIO26/SDIO_DAT2), SW1.1
- net GND: now also J1.14 (GND), J1.20 (GND), J1.25 (GND), J1.30 (GND), J1.34 (GND), J1.39 (GND), J1.9 (GND)

Commit message: 12/18 基板発注
Parts:
- added C15: CC0603KRX7R9BB104, Capacitor_SMD:C_0402_1005Metric, symbol Device:C_Small
- added C16: CL05B104KO5NNNC, Capacitor_SMD:C_0402_1005Metric, symbol Device:C_Small
- added H3, H4, H5, H6: M2 mounting hole, MountingHole:MountingHole_2.2mm_M2, symbol Mechanical:MountingHole
- added J5, J6: EncSide, Library:EncoderPad, symbol Connector:Conn_01x06_Male
- added J7: B2B-XH, Connector_JST:JST_XH_B2B-XH-AM_1x02_P2.50mm_Vertical, symbol Connector_Generic:Conn_01x02
- added U10, U9: AS5047D, Package_SO:TSSOP-14_4.4x5mm_P0.65mm, symbol Sensor_Magnetic:AS5047D
Connections:
- net BTN_DOWN: now also J1.3 (SDA_I2C1/GPIO02); no longer J1.7 (GPCLK0/GPIO04)
- net BTN_LEFT: now also J1.7 (GPCLK0/GPIO04); no longer J1.3 (SDA_I2C1/GPIO02)
- net BTN_RIGHT: now also J1.11 (GPIO17/SPI1_~{CE1}); no longer J1.5 (SCL_I2C1/GPIO03)
- net BTN_UP: now also J1.5 (SCL_I2C1/GPIO03); no longer J1.11 (GPIO17/SPI1_~{CE1})
- net GND: now also J7.1 (Pin_1)
- net +5V: now reaches J1.2 (5V)
- net +5V: now also J1.4 (5V), J7.2 (Pin_2)
- new net: J5.6 (Pin_6), U9.1 (~{CS})
- new net: C15.2, J5.1 (Pin_1), U9.12 (VDD3V3)
- new net: C15.1, J5.2 (Pin_2), U9.13 (GND), U9.5 (TST)
- new net: J5.5 (Pin_5), U9.2 (CLK)
- new net: J5.4 (Pin_4), U9.3 (MISO)
- new net: J5.3 (Pin_3), U9.4 (MOSI)
- new net: J6.6 (Pin_6), U10.1 (~{CS})
- new net: C16.2, J6.1 (Pin_1), U10.12 (VDD3V3)
- new net: C16.1, J6.2 (Pin_2), U10.13 (GND), U10.5 (TST)
- new net: J6.5 (Pin_5), U10.2 (CLK)
- new net: J6.4 (Pin_4), U10.3 (MISO)
- new net: J6.3 (Pin_3), U10.4 (MOSI)
- no-connect marks 4 -> 18
Other:
- note added: "Encoders"
- moved on the sheet: D1, D2, D3, D4, J3, J4, Q1, Q2, Q3, Q4
