File: elec/sub_boards/sub_boards.kicad_pcb (KiCad board)
At the start: 2 copper layers, 84 x 108 mm, 29 parts, among them J1 Raspberry_Pi_5, J3 2.54mm PinHeader, J4 2.54mm PinHeader, J5 EncSide, J6 EncSide, J7 B2B-XH, Q1 ST-1KL3A, Q2 ST-1KL3A, Q3 ST-1KL3A, Q4 ST-1KL3A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

Commit message: サブボード（IFボード）を修正
Signed-off-by: Kazuki Iida <elkel53930@gmail.com>
Parts:
- removed J7: B2B-XH, Connector_JST:JST_XH_B2B-XH-AM_1x02_P2.50mm_Vertical
- moved J1 2.54 mm to (196.8, 124.1)
Connections:
- J1 pad 2: /+5V -> unconnected-(J1-5V-Pad2)
- J1 pad 4: /+5V -> unconnected-(J1-5V-Pad4)
Routing:
- net /CS: track 52.4 -> 63.4 mm
- net /+5V: track 10.2 -> 0.00 mm
- net /MOSI: track 56.7 -> 64.1 mm
- net /BTN_UP: track 28.7 -> 21.6 mm
- net /BTN_DOWN: track 27.2 -> 23.5 mm, vias 1 -> 3
- net /DC: track 56.4 -> 58.3 mm
- net /BTN_RIGHT: track 64.6 -> 63.4 mm, vias 1 -> 2
- net /BTN_LEFT: track 55.1 -> 53.9 mm
- net /SCLK: track 60.6 -> 59.5 mm
- net +3.3V: track 37.0 -> 36.3 mm, vias 1 -> 0
- net /RES: track 65.9 -> 65.7 mm, vias 2 -> 0
- net GND: vias 16 -> 32
Other:
- board text removed: "+5V"
- board text removed: "GND"
