File: elec/main_board/main_board.kicad_pcb (KiCad board)
At the start: 2 copper layers, 84 x 114 mm, 109 parts, among them J1 Conn_01x02, J10 Conn_01x02, J11 B2B-XH-A(LF)(SN), J12 B2B-XH-A(LF)(SN), J16 B4B-ZR(LF)(SN), J2 Conn_01x02, J3 2.54mm PinHeader, J5 B6B-ZR, J6 2.54mm PinHeader, J8 B6B-ZR, J9 MJ-179PH, Q1 IRLML6344, Q2 IRLML6344, Q3 IRLML6344, Q4 IRLML6344, Q5 DMT6008LFG, Q6 DMT6008LFG, Q7 DTC114E, Q8 DTC114E, SW1 SS-22SBH2, U1 ADCS7476, U11 LSM6DSR, U12 OKL-T/6-W12N-C, U13 XC6221B332MR, U14 LM74700QDBVRQ1, U15 MCP73213T-A6SI/MF, U16 LM74700QDBVRQ1, U17 FT231XQ-R, U2 BD63573NUV, U3 ADCS7476, U4 ADCS7476, U5 BD63573NUV, U6 ESP32-S3-WROOM-1, U7 ADCS7476, U8 ADCS7476

Commit message: 回路図更新
・壁センサLEDの抵抗値を100Ωに変更
・電源スイッチを削除
・ESP32のENにプルアップ追加

Signed-off-by: Kazuki Iida <elkel53930@gmail.com>
Parts:
- removed SW1: SS-22SBH2, Library:SS-22SBH2
- added R23: 0603WAF1001T5E, Resistor_SMD:R_0603_1608Metric, F.Cu at (150.4, 40.6)
- R10, R11, R12, R13: value 0603WAF4700T5E -> 0603WAF1000T5E
Connections:
- U14 pad 3: Net-(U14-EN) -> /Power/EXT_PWR
- U16 pad 3: Net-(U16-EN) -> Net-(BT1-+)
Routing:
- net Net-(U14-EN): track 41.2 -> 0.00 mm, vias 1 -> 0
- net /Power/EXT_PWR: track 59.6 -> 21.3 mm, vias 1 -> 0
- net Net-(U16-EN): track 28.1 -> 0.00 mm, vias 1 -> 0
- net Net-(BT1-+): track 26.6 -> 3.62 mm, vias 1 -> 0
- net +3V3: track 286.4 -> 290.1 mm
- net CHIP_PU: track 97.8 -> 99.9 mm
- net /LS_CS: track 22.0 -> 20.4 mm
- net /LF_CS: track 16.2 -> 14.6 mm
- net /LS_EN: track 26.4 -> 25.2 mm
- net /LF_EN: track 29.1 -> 28.3 mm
Other:
- outline, holes or cut-outs redrawn
