File: elec/main_board/main_board.kicad_sch (KiCad schematic)
At the start: 65 parts, among them J1 Conn_01x02, J2 Conn_01x02, J3 2.54mm PinHeader, J5 B6B-ZR, J6 2.54mm PinHeader, J8 B6B-ZR, Q1 IRLML6344, Q2 IRLML6344, Q3 IRLML6344, Q4 IRLML6344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

Commit message: 回路図更新
・壁センサLEDの抵抗値を100Ωに変更
・電源スイッチを削除
・ESP32のENにプルアップ追加

Signed-off-by: Kazuki Iida <elkel53930@gmail.com>
Parts:
- added R23: 0603WAF1001T5E, Resistor_SMD:R_0603_1608Metric, symbol Device:R
- R10, R11, R12, R13: value 0603WAF4700T5E -> 0603WAF1000T5E
Connections:
- net +3V3: now also R23.1
- net CHIP_PU: now also R23.2
Other:
- moved on the sheet: C8, C9
